File: eagle/garage_monitor.brd (EAGLE design)
At the start: 56.8 x 49.5 mm, 20 parts, among them J2 POWER_JACKPTH, T1 2N2222, U1 RELAY-SOLIDSTATEPTH, U2 ATMEGA328P_PDIP

Commit message: updated eagle schematic
Parts:
- Q1: device adafruit:HC33U-V -> crystal:HC49/S
- moved C3 6.35 mm to (21.6, 59.7)
- moved Q1 2.54 mm to (22.9, 52.1)
Routing:
- net GND: track 0.00 -> 165.3 mm
- net VCC: track 0.00 -> 126.5 mm
- net N$18: track 0.00 -> 53.9 mm
- net N$1: track 0.00 -> 53.2 mm
- net RESET: track 0.00 -> 41.8 mm
- net TXMOTION: track 0.00 -> 39.5 mm
- net MOSI: track 0.00 -> 38.2 mm
- net MISO: track 0.00 -> 32.1 mm
- net SCK: track 0.00 -> 32.1 mm
- net DTR: track 0.00 -> 18.3 mm, vias 0 -> 1
- net RXRELAY: track 0.00 -> 17.7 mm
- net N$9: track 0.00 -> 16.5 mm
- net N$2: track 0.00 -> 15.2 mm
- net N$3: track 0.00 -> 14.3 mm
- net N$10: track 0.00 -> 13.9 mm
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