File: eagle/garage_monitor.sch (EAGLE design)
At the start: 20 parts, among them J2 POWER_JACKPTH, T1 2N2222, U1 RELAY-SOLIDSTATEPTH, U2 ATMEGA328P_PDIP

Commit message: updated eagle schematic
Parts:
- Q1: device adafruit:CRYSTALHC33U-V -> crystal:CRYSTALHC49S
Changed lines of the file:
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@@
 <part name="SUPPLY7" library="SparkFun-Aesthetics" deviceset="VCC" device=""/>
 <part name="R2" library="SparkFun-Resistors" deviceset="RESISTOR" device="PTH-1/4W"/>
-<part name="Q1" library="adafruit" deviceset="CRYSTAL" device="HC33U-V"/>
 <part name="C3" library="SparkFun-Capacitors" deviceset="CAP" device="EZ"/>
 <part name="C4" library="SparkFun-Capacitors" deviceset="CAP" device="EZ"/>
@@
 <part name="T1" library="transistor" deviceset="2N2222" device=""/>
 <part name="SUPPLY2" library="SparkFun-Aesthetics" deviceset="VCC" device=""/>
+<part name="Q1" library="crystal" deviceset="CRYSTAL" device="HC49S"/>
 </parts>
 <sheets>
@@
 <instance part="SUPPLY7" gate="1" x="152.4" y="-12.7" rot="R180"/>
 <instance part="R2" gate="G$1" x="152.4" y="-7.62" rot="R90"/>
-<instance part="Q1" gate="G$1" x="66.04" y="43.18" rot="R90"/>
 <instance part="C3" gate="G$1" x="58.42" y="48.26" rot="R90"/>
 <instance part="C4" gate="G$1" x="58.42" y="40.64" rot="R90"/>
@@
 <instance part="T1" gate="G$1" x="0" y="50.8"/>
 <instance part="SUPPLY2" gate="1" x="-10.16" y="63.5" rot="R90"/>
+<instance part="Q1" gate="G$1" x="66.04" y="43.18" rot="R90"/>
 </instances>
 <busses>
@@
 <segment>
 <pinref part="U2" gate="G$1" pin="PB6(XTAL1/TOSC1)"/>
-<pinref part="Q1" gate="G$1" pin="2"/>
 <wire x1="66.04" y1="45.72" x2="66.04" y2="48.26" width="0.1524" layer="91"/>
-<junction x="66.04" y="45.72"/>
 <pinref part="C3" gate="G$1" pin="2"/>
 <wire x1="66.04" y1="48.26" x2="60.96" y2="48.26" width="0.1524" layer="91"/>
+<pinref part="Q1" gate="G$1" pin="2"/>
+<junction x="66.04" y="45.72"/>
 </segment>
 </net>
@@
 <segment>
 <pinref part="U2" gate="G$1" pin="PB7(XTAL2/TOSC2)"/>
-<pinref part="Q1" gate="G$1" pin="1"/>
 <pinref part="C4" gate="G$1" pin="2"/>
 <wire x1="66.04" y1="40.64" x2="60.96" y2="40.64" width="0.1524" layer="91"/>
+<pinref part="Q1" gate="G$1" pin="1"/>
 <junction x="66.04" y="40.64"/>
 </segment>
